Commit message: Promote stable build to main branch

File: tr_description/urdf/amr_body.urdf.xacro (robot description, xacro)
@@ -59,5 +59,5 @@
         </inertial>
         <visual name="lidar_front_visual">
-            <origin xyz="0.0 0.0 0.04" rpy="3.1416 -0.0 0.0" />
+            <origin xyz="0.0 0.0 0.04" rpy="3.1416 0.0 0.0" />
             <geometry>
                 <mesh filename="package://tr_description/meshes/lidar_front.stl" scale="0.001 0.001 0.001" />
@@ -65,5 +65,5 @@
         </visual>
         <collision name="lidar_front_collision">
-            <origin xyz="0.0 0.0 0.04" rpy="3.1416 -0.0 0.0" />
+            <origin xyz="0.0 0.0 0.04" rpy="3.1416 0.0 0.0" />
             <geometry>
                 <mesh filename="package://tr_description/meshes/lidar_front.stl" scale="0.001 0.001 0.001" />
@@ -72,5 +72,5 @@
     </link>
     <joint name="lidar_front_joint" type="fixed">
-        <origin xyz="0.352 0.226 0.04" rpy="3.1416 0.0 0.7854" />
+        <origin xyz="0.352 0.226 0.04" rpy="0.0 0.0 0.7854" />
         <parent link="base_link" />
         <child link="lidar_front" />
@@ -96,7 +96,13 @@
     </link>
     <joint name="lidar_rear_joint" type="fixed">
-        <origin xyz="-0.352 -0.226 0.04" rpy="3.1416 -0.0 0.7854" />
+        <origin xyz="-0.352 -0.226 0.04" rpy="0.0 0.0 0.7854" />
         <parent link="base_link" />
         <child link="lidar_rear" />
+    </joint>
+    <link name="imu_link"/>
+    <joint name="imu_joint" type="fixed">
+        <parent link="base_link"/>
+        <child link="imu_link"/>
+        <origin xyz="0.189 -0.041 0.094" rpy="0 0 0"/>
     </joint>
     <link name="wheel_bogie_right">
@@ -178,14 +184,4 @@
         <axis xyz="0.0 0.0 -1.0" />
     </joint>
-    <transmission name="wheel_left_joint_transmission">
-        <type>transmission_interface/SimpleTransmission</type>
-        <joint name="wheel_left_joint">
-            <hardwareInterface>VelocityJointInterface</hardwareInterface>
-        </joint>
-        <actuator name="wheel_left_joint_motor">
-            <hardwareInterface>VelocityJointInterface</hardwareInterface>
-            <mechanicalReduction>1</mechanicalReduction>
-        </actuator>
-    </transmission>
     <link name="wheel_right">
         <inertial>
@@ -214,14 +210,4 @@
         <axis xyz="0.0 0.0 1.0" />
     </joint>
-    <transmission name="wheel_right_joint_transmission">
-        <type>transmission_interface/SimpleTransmission</type>
-        <joint name="wheel_right_joint">
-            <hardwareInterface>VelocityJointInterface</hardwareInterface>
-        </joint>
-        <actuator name="wheel_right_joint_motor">
-            <hardwareInterface>VelocityJointInterface</hardwareInterface>
-            <mechanicalReduction>1</mechanicalReduction>
-        </actuator>
-    </transmission>
     <link name="caster_fork_front_left">
         <inertial>

File: tr_description/urdf/amr_gazebo.urdf.xacro (robot description, xacro)
@@ -19,5 +19,5 @@
         noise_mean="0.0"
         noise_stddev="0.01"
-        topic_name="scan"
+        topic_name="scan1"
         visualize="false"
     />
@@ -56,3 +56,101 @@
         </plugin>
     </gazebo>
+    <gazebo reference="imu_link">
+        <sensor name="imu_sensor" type="imu">
+            <always_on>true</always_on>
+            <update_rate>100</update_rate>
+            <visualize>false</visualize>
+            <plugin filename="libgazebo_ros_imu_sensor.so" name="gazebo_ros_imu_sensor">
+                <namespace>/</namespace>
+                <topic_name>raw_imu</topic_name> <frame_name>imu_link</frame_name>
+                <initial_orientation_as_reference>false</initial_orientation_as_reference>
+            </plugin>
+            <imu>
+                <angular_velocity>
+                    <x>
+                        <noise type="gaussian">
+                            <mean>0.0</mean>
+                            <stddev>2e-4</stddev>
+                            <bias_mean>0.0000075</bias_mean>
+                            <bias_stddev>0.0000008</bias_stddev>
+                        </noise>
+                    </x>
+                    <y>
+                        <noise type="gaussian">
+                            <mean>0.0</mean>
+                            <stddev>2e-4</stddev>
+                            <bias_mean>0.0000075</bias_mean>
+                            <bias_stddev>0.0000008</bias_stddev>
+                        </noise>
+                    </y>
+                    <z>
+                        <noise type="gaussian">
+                            <mean>0.0</mean>
+                            <stddev>2e-4</stddev>
+                            <bias_mean>0.0000075</bias_mean>
+                            <bias_stddev>0.0000008</bias_stddev>
+                        </noise>
+                    </z>
+                </angular_velocity>
+                <linear_acceleration>
+                    <x>
+                        <noise type="gaussian">
+                            <mean>0.0</mean>
+                            <stddev>1.7e-2</stddev>
+                            <bias_mean>0.1</bias_mean>
+                            <bias_stddev>0.001</bias_stddev>
+                        </noise>
+                    </x>
+                    <y>
+                        <noise type="gaussian">
+                            <mean>0.0</mean>
+                            <stddev>1.7e-2</stddev>
+                            <bias_mean>0.1</bias_mean>
+                            <bias_stddev>0.001</bias_stddev>
+                        </noise>
+                    </y>
+                    <z>
+                        <noise type="gaussian">
+                            <mean>0.0</mean>
+                            <stddev>1.7e-2</stddev>
+                            <bias_mean>0.1</bias_mean>
+                            <bias_stddev>0.001</bias_stddev>
+                        </noise>
+                    </z>
+                </linear_acceleration>
+            </imu>
+        </sensor>
+    </gazebo>
+    <gazebo reference="caster_wheel_front_left">
+        <mu1>0.01</mu1>
+        <mu2>0.01</mu2>
+        <kp>1000000.0</kp>
+        <kd>100.0</kd>
+        <minDepth>0.001</minDepth>
+        <maxVel>1.0</maxVel>
+    </gazebo>
+        <gazebo reference="caster_wheel_front_right">
+        <mu1>0.01</mu1>
+        <mu2>0.01</mu2>
+        <kp>1000000.0</kp>
+        <kd>100.0</kd>
+        <minDepth>0.001</minDepth>
+        <maxVel>1.0</maxVel>
+    </gazebo>
+    <gazebo reference="caster_wheel_rear_left">
+        <mu1>0.01</mu1>
+        <mu2>0.01</mu2>
+        <kp>1000000.0</kp>
+        <kd>100.0</kd>
+        <minDepth>0.001</minDepth>
+        <maxVel>1.0</maxVel>
+    </gazebo>
+    <gazebo reference="caster_wheel_rear_right">
+        <mu1>0.01</mu1>
+        <mu2>0.01</mu2>
+        <kp>1000000.0</kp>
+        <kd>100.0</kd>
+        <minDepth>0.001</minDepth>
+        <maxVel>1.0</maxVel>
+    </gazebo>
 </robot>
